Commit message: ex03

File: ex02/robot.urdf (robot description, URDF)
Before this commit: robot robot, 26 links, 25 joints
Links:
- added link caster_cylinder_link; visual cylinder length=0.1 radius=0.01
- added link left_wheel_cylinder_link; visual cylinder length=0.1 radius=0.01
- added link right_wheel_cylinder_link; visual cylinder length=0.1 radius=0.01
- link back_left_leg: mass None -> 0.125
- link back_right_leg: mass None -> 0.125
- link back_side: mass None -> 0.2
- link body_link: mass None -> 0.5
- link bottom_link: mass None -> 1
- link caster_wheel_link: mass None -> 0.005; geometry collision sphere radius=0.02; visual sphere radius=0.02
- link front_left_leg: mass None -> 0.125
- link front_right_leg: mass None -> 0.125
- link front_side: mass None -> 0.2
- link head_link: mass None -> 0.16666666666666666
- link left_paddle: geometry visual box size=0.02 0.04 0.32
- link left_paddle_plate: geometry visual box size=0.02 0.10 0.14
- link left_side: mass None -> 0.4
- link left_wheel_link: mass None -> 0.1
- link nose_link: mass None -> 0.05
- link right_paddle: geometry visual box size=0.02 0.04 0.32
- link right_paddle_plate: geometry visual box size=0.02 0.10 0.14
- link right_side: mass None -> 0.4
- link right_wheel_link: mass None -> 0.1
Joints:
- added joint caster_cylinider_joint: type fixed, parent caster_wheel_link, child caster_cylinder_link, origin xyz=0.1 0 0 rpy=0 1.5707963267948966 0
- added joint left_wheel_cylinider_joint: type fixed, parent left_wheel_link, child left_wheel_cylinder_link, origin xyz=0.1 0 0 rpy=0 1.5707963267948966 0
- added joint right_wheel_cylinider_joint: type fixed, parent right_wheel_link, child right_wheel_cylinder_link, origin xyz=0.1 0 0 rpy=0 1.5707963267948966 0
- joint caster_wheel_joint: axis 1 1 1 -> (none); origin xyz=0.16 0 -0.04 rpy=0 0 0 -> xyz=-0.16 0 -0.06 rpy=0 0 0; type continuous -> fixed
- joint left_wheel_joint: axis 0 0 1 -> 0 0 1.0; origin xyz=-0.12 0.21 0 rpy=-1.5707963267948966 0 0 -> xyz=0.1 0.215 0 rpy=-1.5707963267948966 0 0
- joint pig_joint: origin xyz=0.02 0 0.20 rpy=0 0 0 -> xyz=-0.02 0 0.20 rpy=0 0 0
- joint right_wheel_joint: axis 0 0 1 -> 0 0 -1.0; origin xyz=-0.12 -0.21 0 rpy=-1.5707963267948966 0 0 -> xyz=0.1 -0.215 0 rpy=1.5707963267948966 0 0
